File: TTL/Принципиальная/принципиальная.sch (KiCad schematic (older format))
At the start: 29 parts

Commit message: Upd
Other:
- note added: "MCLK"
- note added: "VCC"
Changed lines of the file:
@@
 Wire Bus Line
 	11450 2050 11450 8250
+Text Notes 3550 5700 0    50   ~ 0
+VCC
+Text Notes 3550 5800 0    50   ~ 0
+GND
+Text Notes 3550 7050 0    50   ~ 0
+MCLK
+Text Notes 3550 7250 0    50   ~ 0
+GND
 $EndSCHEMATC
